File: amp_controller.kicad_sch (KiCad schematic)
At the start: 50 parts, among them Q1 BC848, Q2 BC848, Q3 BC848, U1 RaspberryPi_Pico_W, U2 TSR_1-2450, U3 LT1175-5_SOT223, U4 LM4040DBZ-3, U6 EL3H7(C)(TA)-G, U7 MCP1700x-330xxTT, U8 LM2904

Commit message: passing DRC check, op amp input issue fixed
Parts:
- added FB3: FerriteBead, Inductor_SMD:L_0805_2012Metric, symbol Device:FerriteBead
- added TP-PEAK1, TP-VREF1, TPG1: TestPoint, TestPoint:TestPoint_THTPad_1.0x1.0mm_Drill0.5mm, symbol Connector:TestPoint
- Q1, Q2, Q3: footprint Package_TO_SOT_SMD:SOT-23 -> Package_TO_SOT_SMD:SOT-723
Connections:
- net +5V: no longer U7.3 (VI)
- net ADC_VREF: now also TP-VREF1.1
- net GND: now also GPIO16,17.1 (Pin_1), FB3.2, TPG1.1; no longer C2.2, GPIO16,17.3 (Pin_3), R10.2, R11.2, R8.2, U1.33 (AGND), U4.2 (A), Z1.2 (A)
- net PEAK: now also TP-PEAK1.1
- net VSYS: now also U7.3 (VI)
- net at C3.2, R10.1: now also U8.2 (-); no longer U8.3 (+)
- net at U1.21 (GPIO16): now also GPIO16,17.3 (Pin_3); no longer GPIO16,17.1 (Pin_1)
- net at R8.1, R9.1: now also U8.3 (+); no longer U8.2 (-)
- net at D3.2 (A), R6.2, R7.1: now also U8.6 (-); no longer U8.5 (+)
- net at R11.1: now also U8.5 (+); no longer U8.6 (-)
- new net AGND: C2.2, FB3.1, R10.2, R11.2, R8.2, U1.33 (AGND), U4.2 (A), Z1.2 (A)
Other:
- note added: "Music input peak detector. Signal is buffered and amplified by 20dB to overcome the noise limitations of the Pico ADC which is only 8.7ENOB or ~60dB. Using the amplified signal moves the detection limit down to -80dB. The signal is then half wave rectified and averaged with C2 in parallel with the 100k load of the Pico ADC. Zener D5 limits the voltage input to the ADC to 2.4V, so around 100mV RMS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"
- note removed: "Music input peak detector. Signal is buffered and amplified by 20dB to overcome the noise limitations of the Pico ADC which is only 8.7ENOB or ~60dB. Using the amplified signal moves the detection limit down to -80dB. The signal is then half wave rectified and averaged with C2 in parallel with the 100k load of the Pico ADC. Zener D5 limits the voltage input to the ADC to 2.5V"
- moved on the sheet: C2, C3, D2, D3, GPIO16,17, MUSIC_IN1, MUSIC_THRU1, R10, R11, R6, R7, R8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

Commit message: tweaked layout and music sense resistors
Parts:
- added C5: 1u, Capacitor_SMD:C_0805_2012Metric, symbol Device:C
- added J1: Conn_01x02_Pin, Connector_PinHeader_2.54mm:PinHeader_1x02_P2.54mm_Vertical, symbol Connector:Conn_01x02_Pin
- added TPAG1: TestPoint, TestPoint:TestPoint_THTPad_1.0x1.0mm_Drill0.5mm, symbol Connector:TestPoint
- added U5: ADS1110, Package_TO_SOT_SMD:SOT-23-6, symbol Analog_ADC:ADS1110
- D1, D4: value 1N5819WS -> D_Schottky; footprint Diode_SMD:D_SOD-323 -> Diode_SMD:D_SOD-523; symbol Diode:1N5819WS -> Device:D_Schottky; LCSC C2480 -> C145179
- D2, D3: value 1N5819WS -> D_Schottky; footprint Diode_SMD:D_SOD-323 -> Diode_SMD:D_SOD-523; symbol Diode:1N5819WS -> Device:D_Schottky; LCSC C2128 -> C145179
- R10: value 90k -> 91k; LCSC C5123603 -> C2930321
- R6, R7: value 10k -> 1M; LCSC C17414 -> C17514
- R8: value 10k -> 100k; LCSC C17414 -> C149504
- R9: value 100k -> 1M; LCSC C149504 -> C17514
- renumbered GPIO2,3 to GPIO3,2,G1, TP-VREF1 to TPVR1
Connections:
- net +5V: now also C5.2, U5.5 (VDD)
- net AGND: now also TPAG1.1, U5.6 (VIN-)
- net GND: now also C5.1, U5.2 (GND)
- net PEAK: now also U5.1 (VIN+)
- net GPIO17: now reaches GPIO16,17.2 (Pin_2), U1.22 (GPIO17)
- net GPIO16: now reaches GPIO16,17.3 (Pin_3), U1.21 (GPIO16)
- net I2C1_SDA: now reaches U1.31 (GPIO26_ADC0)
- net I2C1_SDA: now also U5.4 (SDA)
- net I2C1_SCL: now reaches U1.32 (GPIO27_ADC1)
- net I2C1_SCL: now also U5.3 (SCL)
- net at R8.1, R9.1, U8.3 (+): now also J1.2 (Pin_2)
- net at R6.1, R9.2, U8.1: now also J1.1 (Pin_1)
Other:
- moved on the sheet: R8, R9
